File: Hardware/Electronics/IRIS.brd (EAGLE design)
At the start: 55.9 x 15.2 mm, 3 parts, among them X1 MINI-USB-32005-201

Commit message: Schematic modifications…
Parts:
- removed U$1: TCD1304AP, SPectrolib:TCD1304AP
- removed U$2: AT32UC3C, SPectrolib:TQFP64
- removed X1: MINI-USB-32005-201, con-cypressindustries:32005-201
- added JP1: (no value), jumper:JP1
- added U1: AT32UC3C, IRIS:TQFP64
- added U2: TCD1304AP, IRIS:TCD1304AP
- added X2: MINI-USB-32005-201, con-cypressindustries:32005-201
Connections:
- removed net CCD: U$1.P$21, U$2.P$2
- removed net N$3: U$1.P$5, U$2.P$37
- new net ADCIN0: JP1.2, U1.P$7
- new net OS: JP1.1, U2.P$21
- new net TC0A2: U1.P$38, U2.P$5
- new net TC0B1: U1.P$37, U2.P$4
- new net TC1B1: U1.P$34, U2.P$3
- new net TCK: U1.P$1
- new net TDI: U1.P$2
- new net TDO: U1.P$3
- new net TMS: U1.P$4
- new net VAD: U2.P$2
- new net VCC: U1.P$18, U1.P$23, U1.P$27, U1.P$35, U1.P$5, U1.P$51, X2.1
- new net VDD: U2.P$1
- new net XIN0: U1.P$31
- new net XOUT0: U1.P$32
- net GND: now also U1.P$17, U1.P$26, U1.P$30, U1.P$36, U1.P$52, U1.P$6, U2.P$22, X2.4, X2.5; no longer U$2.P$1, U$2.P$10, U$2.P$5, U$2.P$6, U$2.P$7, U$2.P$8, U$2.P$9
- net N$1: now also U1.P$24, X2.2; no longer U$1.P$3, U$2.P$39
- net N$2: now also U1.P$25, X2.3; no longer U$1.P$4, U$2.P$38
Other:
- board outline removed
Changed lines of the file:
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@@
 <setting verticaltext="up"/>
 </settings>
-<grid distance="1" unitdist="mm" unit="mm" style="lines" multiple="1" display="no" altdistance="0.025" altunitdist="inch" altunit="inch"/>
+<grid distance="0.05" unitdist="inch" unit="inch" style="lines" multiple="1" display="no" altdistance="0.025" altunitdist="inch" altunit="inch"/>
 <layers>
 <layer number="1" name="Top" color="4" fill="1" visible="yes" active="yes"/>
@@
 <board>
 <plain>
-<wire x1="0" y1="0" x2="55.86" y2="0" width="0" layer="20"/>
-<wire x1="55.86" y1="0" x2="55.86" y2="15.18" width="0" layer="20"/>
-<wire x1="55.86" y1="15.18" x2="0" y2="15.18" width="0" layer="20"/>
-<wire x1="0" y1="15.18" x2="0" y2="0" width="0" layer="20"/>
 </plain>
 <attributes>
@@
 </autorouter>
 <elements>
-<element name="U$1" library="SPectrolib" package="TCD1304AP" value="TCD1304AP" x="20.32" y="7.62"/>
-<element name="U$2" library="SPectrolib" package="TQFP64" value="AT32UC3C" x="39.63" y="7.38" rot="R180"/>
-<element name="X1" library="con-cypressindustries" package="32005-201" value="MINI-USB-32005-201" x="50.8" y="7.62" rot="R180">
-<attribute name="OC_NEWARK" value="unknown" x="50.8" y="7.62" size="1.778" layer="27" rot="R180" display="off"/>
-<attribute name="MPN" value="" x="50.8" y="7.62" size="1.778" layer="27" rot="R180" display="off"/>
-<attribute name="MF" value="" x="50.8" y="7.62" size="1.778" layer="27" rot="R180" display="off"/>
-<attribute name="OC_FARNELL" value="unknown" x="50.8" y="7.62" size="1.778" layer="27" rot="R180" display="off"/>
+<element name="U1" library="IRIS" package="TQFP64" value="AT32UC3C" x="-11.43" y="-31.75"/>
+<element name="U2" library="IRIS" package="TCD1304AP" value="TCD1304AP" x="8.89" y="-31.75"/>
+<element name="X2" library="con-cypressindustries" package="32005-201" value="MINI-USB-32005-201" x="-24.13" y="-31.75">
+<attribute name="OC_NEWARK" value="unknown" x="-24.13" y="-31.75" size="1.778" layer="27" display="off"/>
+<attribute name="MPN" value="" x="-24.13" y="-31.75" size="1.778" layer="27" display="off"/>
+<attribute name="MF" value="" x="-24.13" y="-31.75" size="1.778" layer="27" display="off"/>
+<attribute name="OC_FARNELL" value="unknown" x="-24.13" y="-31.75" size="1.778" layer="27" display="off"/>
 </element>
+<element name="JP1" library="jumper" package="JP1" value="" x="-34.29" y="-35.56"/>
 </elements>
 <signals>
 <signal name="GND">
-<contactref element="U$2" pad="P$7"/>
-<contactref element="U$2" pad="P$8"/>
-<contactref element="U$2" pad="P$9"/>
-<contactref element="U$2" pad="P$5"/>
-<contactref element="U$2" pad="P$6"/>
-<contactref element="U$2" pad="P$10"/>
-<contactref element="U$2" pad="P$1"/>
-<wire x1="45.13" y1="5.63" x2="45.13" y2="3.63" width="0" layer="19" extent="1-1"/>
-<wire x1="45.13" y1="6.13" x2="45.13" y2="5.63" width="0" layer="19" extent="1-1"/>
-<wire x1="45.13" y1="6.63" x2="45.13" y2="6.13" width="0" layer="19" extent="1-1"/>
-<wire x1="45.13" y1="7.13" x2="45.13" y2="6.63" width="0" layer="19" extent="1-1"/>
-<wire x1="45.13" y1="7.63" x2="45.13" y2="7.13" width="0" layer="19" extent="1-1"/>
-<wire x1="45.13" y1="8.13" x2="45.13" y2="7.63" width="0" layer="19" extent="1-1"/>
+<contactref element="U1" pad="P$26"/>
+<contactref element="U1" pad="P$6"/>
+<contactref element="U1" pad="P$36"/>
+<contactref element="U1" pad="P$52"/>
+<contactref element="U1" pad="P$17"/>
+<contactref element="U1" pad="P$30"/>
+<contactref element="X2" pad="4"/>
+<contactref element="X2" pad="5"/>
+<contactref element="U2" pad="P$22"/>
+<wire x1="-21.13" y1="-32.55" x2="-21.13" y2="-33.35" width="0" layer="19" extent="1-1"/>
+<wire x1="-15.18" y1="-37.25" x2="-21.13" y2="-32.55" width="0" layer="19" extent="1-1"/>
+<wire x1="-10.68" y1="-37.25" x2="-15.18" y2="-37.25" width="0" layer="19" extent="1-1"/>
+<wire x1="-8.68" y1="-37.25" x2="-10.68" y2="-37.25" width="0" layer="19" extent="1-1"/>
+<wire x1="-3.81" y1="-26.67" x2="-8.68" y2="-37.25" width="0" layer="19" extent="1-1"/>
+<wire x1="-5.93" y1="-34" x2="-8.68" y2="-37.25" width="0" layer="19" extent="1-1"/>
+<wire x1="-16.93" y1="-30.5" x2="-15.18" y2="-37.25" width="0" layer="19" extent="1-1"/>
+<wire x1="-9.18" y1="-26.25" x2="-5.93" y2="-34" width="0" layer="19" extent="1-1"/>
+</signal>
+<signal name="VCC">
+<contactref element="U1" pad="P$18"/>
+<contactref element="U1" pad="P$5"/>
+<contactref element="U1" pad="P$35"/>
+<contactref element="U1" pad="P$51"/>
+<contactref element="U1" pad="P$27"/>
+<contactref element="U1" pad="P$23"/>
+<contactref element="X2" pad="1"/>
+<wire x1="-12.18" y1="-37.25" x2="-14.68" y2="-37.25" width="0" layer="19" extent="1-1"/>
+<wire x1="-10.18" y1="-37.25" x2="-12.18" y2="-37.25" width="0" layer="19" extent="1-1"/>
+<wire x1="-5.93" y1="-34.5" x2="-10.18" y2="-37.25" width="0" layer="19" extent="1-1"/>
+<wire x1="-16.93" y1="-30" x2="-14.68" y2="-37.25" width="0" layer="19" extent="1-1"/>
+<wire x1="-21.13" y1="-30.15" x2="-16.93" y2="-30" width="0" layer="19" extent="1-1"/>
+<wire x1="-8.68" y1="-26.25" x2="-5.93" y2="-34.5" width="0" layer="19" extent="1-1"/>
 </signal>
 <signal name="N$1">
-<contactref element="U$1" pad="P$3"/>
-<contactref element="U$2" pad="P$39"/>
-<wire x1="12.7" y1="2.54" x2="34.13" y2="8.13" width="0" layer="19" extent="1-1"/>
+<contactref element="U1" pad="P$24"/>
+<contactref element="X2" pad="2"/>
+<wire x1="-11.68" y1="-37.25" x2="-21.13" y2="-30.95" width="0" layer="19" extent="1-1"/>
 </signal>
 <signal name="N$2">
-<contactref element="U$1" pad="P$4"/>
-<contactref element="U$2" pad="P$38"/>
-<wire x1="15.24" y1="2.54" x2="34.13" y2="8.63" width="0" layer="19" extent="1-1"/>
-</signal>
-<signal name="N$3">
-<contactref element="U$1" pad="P$5"/>
-<contactref element="U$2" pad="P$37"/>
-<wire x1="17.78" y1="2.54" x2="34.13" y2="9.13" width="0" layer="19" extent="1-1"/>
-</signal>
-<signal name="CCD">
-<contactref element="U$1" pad="P$21"/>
-<contactref element="U$2" pad="P$2"/>
-<wire x1="10.16" y1="12.7" x2="45.13" y2="4.13" width="0" layer="19" extent="1-1"/>
+<contactref element="U1" pad="P$25"/>
+<contactref element="X2" pad="3"/>
+<wire x1="-11.18" y1="-37.25" x2="-21.13" y2="-31.75" width="0" layer="19" extent="1-1"/>
+</signal>
+<signal name="TCK">
+<contactref element="U1" pad="P$1"/>
+</signal>
+<signal name="TDI">
+<contactref element="U1" pad="P$2"/>
+</signal>
+<signal name="TDO">
+<contactref element="U1" pad="P$3"/>
+</signal>
+<signal name="TMS">
+<contactref element="U1" pad="P$4"/>
+</signal>
+<signal name="XIN0">
+<contactref element="U1" pad="P$31"/>
+</signal>
+<signal name="XOUT0">
+<contactref element="U1" pad="P$32"/>
+</signal>
+<signal name="ADCIN0">
+<contactref element="U1" pad="P$7"/>
+<contactref element="JP1" pad="2"/>
+<wire x1="-16.93" y1="-31" x2="-34.29" y2="-34.29" width="0" layer="19" extent="1-1"/>
+</signal>
+<signal name="OS">
+<contactref element="U2" pad="P$21"/>
+<contactref element="JP1" pad="1"/>
+<wire x1="-1.27" y1="-26.67" x2="-34.29" y2="-36.83" width="0" layer="19" extent="1-1"/>
+</signal>
+<signal name="VDD">
+<contactref element="U2" pad="P$1"/>
+</signal>
+<signal name="VAD">
+<contactref element="U2" pad="P$2"/>
+</signal>
+<signal name="TC1B1">
+<contactref element="U1" pad="P$34"/>
+<contactref element="U2" pad="P$3"/>
+<wire x1="-5.93" y1="-35" x2="1.27" y2="-36.83" width="0" layer="19" extent="1-1"/>
+</signal>
+<signal name="TC0B1">
+<contactref element="U1" pad="P$37"/>
+<contactref element="U2" pad="P$4"/>
+<wire x1="-5.93" y1="-33.5" x2="3.81" y2="-36.83" width="0" layer="19" extent="1-1"/>
+</signal>
+<signal name="TC0A2">
+<contactref element="U1" pad="P$38"/>
+<contactref element="U2" pad="P$5"/>
+<wire x1="-5.93" y1="-33" x2="6.35" y2="-36.83" width="0" layer="19" extent="1-1"/>
 </signal>
 </signals>

Commit message: Board routed.
Parts:
- added C1, C3, C6: 4.7u X7R 1463379, rcl:C0603
- added C10: 100nF, rcl:C0603
- added C11, C2, C4: 1n NPO 1535563, rcl:C0402
- added C17, C18: 4.7u, resistor:C0805
- added C5, C7: 470pF NPO 1301710RL, rcl:C0603
- added C8, C9: 2.2uF X7R 1657930RL, rcl:C0603
- added R1, R2: 39, rcl:R0603
- added R3: 47k, rcl:R0603
- added U$1: AWIRE, IRIS:AWIRE
- moved X2 101.5 mm to (69.4, 7.62), turned to 180 degrees
- moved JP1 87.2 mm to (42.9, 5.08), turned to 180 degrees
- moved U1 73.6 mm to (50.8, 7.62), turned to 90 degrees
- moved U2 41.1 mm to (20.6, 7.62), turned to 180 degrees
Connections:
- new net N$3: R1.2, X2.2
- new net N$4: R2.2, X2.3
- new net RSTN: R3.1, U$1.P$2, U1.P$64
- net GND: now also C1.2, C10.2, C11.2, C17.2, C18.2, C2.2, C3.2, C4.2, C5.2, C6.2, C7.2, C8.2, C9.2, U$1.P$3
- net N$1: now also R1.1; no longer X2.2
- net N$2: now also R2.1; no longer X2.3
- net VCC: now also C1.1, C10.1, C11.1, C2.1, C3.1, C4.1, C5.1, C6.1, C7.1, C8.1, C9.1, R3.2, U$1.P$1
- net VDD: now also C17.1, C18.1
Routing:
- net TC0A2: track 0.00 -> 34.1 mm
- net GND: track 0.00 -> 29.6 mm, vias 0 -> 6
- net TC0B1: track 0.00 -> 28.9 mm
- net TC1B1: track 0.00 -> 28.7 mm, vias 0 -> 1
- net RSTN: track 0.00 -> 23.1 mm, vias 0 -> 2
- net VCC: track 0.00 -> 21.5 mm, vias 0 -> 3
- net OS: track 0.00 -> 13.6 mm
- net ADCIN0: track 0.00 -> 9.55 mm
- net N$1: track 0.00 -> 4.83 mm
- net N$2: track 0.00 -> 4.70 mm
- net VDD: track 0.00 -> 4.31 mm
- net N$4: track 0.00 -> 3.97 mm
- net N$3: track 0.00 -> 3.77 mm
- added copper zone on layer 16, net GND
- added copper zone on layer 1, net VCC
Other:
- board outline added: 74 x 15.6 mm
- board text added: "IRIS v1.0"

Commit message: First candidate for v1.0
Parts:
- added C12, C13: 22pF, rcl:C0402
- added Q2: 12MHz, Forrequi:CRYSTAL-SMD-5X3
- JP1: value (none) -> Output signal
- moved C3 1.24 mm to (53.2, 10.6)
- moved C4 1.24 mm to (53.2, 11.7)
- moved R2 1.06 mm to (62.2, 9.05)
- moved R1 1.06 mm to (62.2, 7.78)
- moved C1 0.95 mm to (42.5, 10.8)
- moved C10 0.95 mm to (54.8, 6.19)
- moved C11 0.95 mm to (43.7, 10.8)
- moved C17 0.95 mm to (34.1, 9.37)
- moved C6 0.95 mm to (48.9, 6.67)
- moved U$1 0.95 mm to (59.1, 3.49)
- moved C2 0.95 mm to (48.9, 5.40)
- moved C5 0.95 mm to (59.1, 5.08)
- moved C8 0.95 mm to (57.8, 5.08)
- moved JP1 0.95 mm to (42.9, 6.03)
- moved R3 0.95 mm to (61.6, 5.08)
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Connections:
- removed net TCK: U1.P$1
- removed net TDI: U1.P$2
- removed net TDO: U1.P$3
- removed net TMS: U1.P$4
- removed net VAD: U2.P$2
- removed net VDD: C17.1, C18.1, U2.P$1
- removed net XIN0: U1.P$31
- removed net XOUT0: U1.P$32
- new net N$21: C12.1, Q2.3, U1.P$31
- new net N$22: C13.1, Q2.1, U1.P$32
- net GND: now also C12.2, C13.2
- net VCC: now also C17.1, C18.1, U2.P$1, U2.P$2
Routing:
- net N$22: track 0.00 -> 8.53 mm, vias 0 -> 1
- net VCC: track 21.5 -> 27.8 mm
- net N$21: track 0.00 -> 5.81 mm, vias 0 -> 1
- net VDD: track 4.31 -> 0.00 mm
- net GND: track 29.6 -> 33.4 mm
- net RSTN: track 23.1 -> 21.5 mm
Other:
- board size 74 x 15.6 mm -> 74 x 17.6 mm

Commit message: First version
Parts:
- removed U$1: AWIRE, IRIS:AWIRE
- added U3: AWIRE, IRIS:AWIRE
- moved C12 1.27 mm to (57.9, 9.37)
- moved C18 1.27 mm to (34.1, 12.9)
- moved C7 1.27 mm to (57.8, 12.2)
- moved C9 1.27 mm to (59.1, 12.2)
- moved C2 1.27 mm to (48.9, 6.67)
- moved JP1 1.27 mm to (42.9, 7.30)
- moved R1 1.27 mm to (62.2, 9.05)
- moved C1 1.27 mm to (42.5, 12.1)
- moved C10 1.27 mm to (54.8, 7.46)
- moved C11 1.27 mm to (43.7, 12.1)
- moved C13 1.27 mm to (57.9, 16.7)
- moved C17 1.27 mm to (34.1, 10.6)
- moved C3 1.27 mm to (53.2, 11.9)
- moved C4 1.27 mm to (53.2, 13.0)
- moved C5 1.27 mm to (59.1, 6.35)
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Connections:
- net GND: now also U3.P$3; no longer U$1.P$3
- net RSTN: now also U3.P$2; no longer U$1.P$2
- net VCC: now also U3.P$1; no longer U$1.P$1
Routing:
- net RSTN: track 21.5 -> 22.6 mm
Other:
- board size 74 x 17.6 mm -> 75 x 19.6 mm
