File: FPGA/PCB/IRIS1304_v3.0.brd (EAGLE design)
At the start: 64 x 87 mm, 74 parts, among them IC2 FT2232H, Q1 ASFL, Q2 ASFL, U2 LT6202IS5PBF, U3 LD1117-33, U4 LD1117-25, U6 ADR3430ARJZ-R2, U7 M93C56-WMN6P, U8 XCF02SVOG20C, U9 LD1117-12, X1 MINI-USB-32005-201

Commit message: v3.0
Parts:
- added GND31: TEST, IRIS lib v1.0:TEST
Connections:
- net GND: now also GND31.P$1
Other:
- board text added: "v4.0"
- board text removed: "v2.23"
Changed lines of the file:
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@@
 <layer number="220" name="220bmp" color="21" fill="1" visible="no" active="no"/>
 <layer number="221" name="221bmp" color="22" fill="1" visible="no" active="no"/>
+<layer number="222" name="222bmp" color="23" fill="1" visible="no" active="no"/>
 <layer number="223" name="223bmp" color="24" fill="1" visible="no" active="no"/>
 <layer number="224" name="224bmp" color="25" fill="1" visible="no" active="no"/>
@@
 <text x="37.1475" y="13.335" size="0.6096" layer="22" rot="MR0">ICG</text>
 <text x="47.625" y="2.2225" size="0.6096" layer="22" rot="MR0">SH</text>
-<text x="31.7627" y="75.16495" size="0.6096" layer="22" rot="MR0">v2.23</text>
+<text x="31.7627" y="75.16495" size="0.6096" layer="22" rot="MR0">v4.0</text>
 <rectangle x1="41.8211" y1="73.9013" x2="42.9641" y2="73.9267" layer="22" rot="R180"/>
 <rectangle x1="41.4147" y1="73.9267" x2="43.1927" y2="73.9521" layer="22" rot="R180"/>
@@
 <attribute name="OC_FARNELL" value="unknown" x="45.72" y="27.94" size="1.778" layer="27" display="off"/>
 </element>
+<element name="GND31" library="IRIS lib v1.0" package="TEST" value="TEST" x="56.03875" y="66.04">
+<attribute name="MPN" value="001-1007-040FB9" x="56.03875" y="66.04" size="0.04" layer="27" display="off"/>
+<attribute name="MF" value="ITT CANNON" x="56.03875" y="66.04" size="0.04" layer="27" display="off"/>
+<attribute name="OC_FARNELL" value="1347797" x="56.03875" y="66.04" size="0.04" layer="27" display="off"/>
+</element>
 </elements>
 <signals>
@@
 <wire x1="32.9175" y1="48.5775" x2="32.9175" y2="47.625" width="0.254" layer="16"/>
 <wire x1="32.86125" y1="48.73625" x2="32.86125" y2="48.63375" width="0.254" layer="16"/>
+<contactref element="GND31" pad="P$1"/>
 </signal>
 <signal name="N$11">
